File: hardware/rev-c-active-shunt/RevC_Active_Controller_v0.3.1.kicad_sch (KiCad schematic)
At the start: 25 parts, among them J1 TEST_A / GND, J2 +12/GND/-12, U1 OPA551PA

Commit message: Rev.C v0.3.1: align TP values and NC parity
Parts:
- TP1: value TEST_A -> TP8
- TP2: value OUT -> TP8
- TP3: value NINV -> TP8
- TP4: value INJ_NODE -> TP8
- TP5: value +12V -> TP8
- TP6: value -12V -> TP8
- TP7: value GND -> TP8
- TP8: value FLAG -> TP8
Changed lines of the file:
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@@
   (symbol (lib_id "RevC:TP1P") (at 20.00 82.00 0) (unit 1)
     (in_bom yes) (on_board yes)
-    (default_instance (reference "TP1") (unit 1) (value "TEST_A") (footprint "TestPoint:TestPoint_THTPad_D1.5mm_Drill0.8mm"))
+    (default_instance (reference "TP1") (unit 1) (value "TP1") (footprint "TestPoint:TestPoint_THTPad_D1.5mm_Drill0.8mm"))
     (property "Reference" "TP1" (id 0) (at 20.00 79.00 0) (effects (font (size 1.0 1.0))))
-    (property "Value" "TEST_A" (id 1) (at 20.00 85.00 0) (effects (font (size 0.9 0.9))))
+    (property "Value" "TP8" (id 1) (at 20.00 85.00 0) (effects (font (size 0.9 0.9))))
     (property "Footprint" "TestPoint:TestPoint_THTPad_D1.5mm_Drill0.8mm" (id 2) (at 20.00 82.00 0) (effects (font (size 1.0 1.0)) hide))
     (property "Datasheet" "~" (id 3) (at 20.00 82.00 0) (effects (font (size 1.0 1.0)) hide))
@@
   (symbol (lib_id "RevC:TP1P") (at 40.00 82.00 0) (unit 1)
     (in_bom yes) (on_board yes)
-    (default_instance (reference "TP2") (unit 1) (value "OUT") (footprint "TestPoint:TestPoint_THTPad_D1.5mm_Drill0.8mm"))
+    (default_instance (reference "TP2") (unit 1) (value "TP2") (footprint "TestPoint:TestPoint_THTPad_D1.5mm_Drill0.8mm"))
     (property "Reference" "TP2" (id 0) (at 40.00 79.00 0) (effects (font (size 1.0 1.0))))
-    (property "Value" "OUT" (id 1) (at 40.00 85.00 0) (effects (font (size 0.9 0.9))))
+    (property "Value" "TP8" (id 1) (at 40.00 85.00 0) (effects (font (size 0.9 0.9))))
     (property "Footprint" "TestPoint:TestPoint_THTPad_D1.5mm_Drill0.8mm" (id 2) (at 40.00 82.00 0) (effects (font (size 1.0 1.0)) hide))
     (property "Datasheet" "~" (id 3) (at 40.00 82.00 0) (effects (font (size 1.0 1.0)) hide))
@@
   (symbol (lib_id "RevC:TP1P") (at 60.00 82.00 0) (unit 1)
     (in_bom yes) (on_board yes)
-    (default_instance (reference "TP3") (unit 1) (value "NINV") (footprint "TestPoint:TestPoint_THTPad_D1.5mm_Drill0.8mm"))
+    (default_instance (reference "TP3") (unit 1) (value "TP3") (footprint "TestPoint:TestPoint_THTPad_D1.5mm_Drill0.8mm"))
     (property "Reference" "TP3" (id 0) (at 60.00 79.00 0) (effects (font (size 1.0 1.0))))
-    (property "Value" "NINV" (id 1) (at 60.00 85.00 0) (effects (font (size 0.9 0.9))))
+    (property "Value" "TP8" (id 1) (at 60.00 85.00 0) (effects (font (size 0.9 0.9))))
     (property "Footprint" "TestPoint:TestPoint_THTPad_D1.5mm_Drill0.8mm" (id 2) (at 60.00 82.00 0) (effects (font (size 1.0 1.0)) hide))
     (property "Datasheet" "~" (id 3) (at 60.00 82.00 0) (effects (font (size 1.0 1.0)) hide))
@@
   (symbol (lib_id "RevC:TP1P") (at 80.00 82.00 0) (unit 1)
     (in_bom yes) (on_board yes)
-    (default_instance (reference "TP4") (unit 1) (value "INJ_NODE") (footprint "TestPoint:TestPoint_THTPad_D1.5mm_Drill0.8mm"))
+    (default_instance (reference "TP4") (unit 1) (value "TP4") (footprint "TestPoint:TestPoint_THTPad_D1.5mm_Drill0.8mm"))
     (property "Reference" "TP4" (id 0) (at 80.00 79.00 0) (effects (font (size 1.0 1.0))))
-    (property "Value" "INJ_NODE" (id 1) (at 80.00 85.00 0) (effects (font (size 0.9 0.9))))
+    (property "Value" "TP8" (id 1) (at 80.00 85.00 0) (effects (font (size 0.9 0.9))))
     (property "Footprint" "TestPoint:TestPoint_THTPad_D1.5mm_Drill0.8mm" (id 2) (at 80.00 82.00 0) (effects (font (size 1.0 1.0)) hide))
     (property "Datasheet" "~" (id 3) (at 80.00 82.00 0) (effects (font (size 1.0 1.0)) hide))
@@
   (symbol (lib_id "RevC:TP1P") (at 100.00 82.00 0) (unit 1)
     (in_bom yes) (on_board yes)
-    (default_instance (reference "TP5") (unit 1) (value "+12V") (footprint "TestPoint:TestPoint_THTPad_D1.5mm_Drill0.8mm"))
+    (default_instance (reference "TP5") (unit 1) (value "TP5") (footprint "TestPoint:TestPoint_THTPad_D1.5mm_Drill0.8mm"))
     (property "Reference" "TP5" (id 0) (at 100.00 79.00 0) (effects (font (size 1.0 1.0))))
-    (property "Value" "+12V" (id 1) (at 100.00 85.00 0) (effects (font (size 0.9 0.9))))
+    (property "Value" "TP8" (id 1) (at 100.00 85.00 0) (effects (font (size 0.9 0.9))))
     (property "Footprint" "TestPoint:TestPoint_THTPad_D1.5mm_Drill0.8mm" (id 2) (at 100.00 82.00 0) (effects (font (size 1.0 1.0)) hide))
     (property "Datasheet" "~" (id 3) (at 100.00 82.00 0) (effects (font (size 1.0 1.0)) hide))
@@
   (symbol (lib_id "RevC:TP1P") (at 120.00 82.00 0) (unit 1)
     (in_bom yes) (on_board yes)
-    (default_instance (reference "TP6") (unit 1) (value "-12V") (footprint "TestPoint:TestPoint_THTPad_D1.5mm_Drill0.8mm"))
+    (default_instance (reference "TP6") (unit 1) (value "TP6") (footprint "TestPoint:TestPoint_THTPad_D1.5mm_Drill0.8mm"))
     (property "Reference" "TP6" (id 0) (at 120.00 79.00 0) (effects (font (size 1.0 1.0))))
-    (property "Value" "-12V" (id 1) (at 120.00 85.00 0) (effects (font (size 0.9 0.9))))
+    (property "Value" "TP8" (id 1) (at 120.00 85.00 0) (effects (font (size 0.9 0.9))))
     (property "Footprint" "TestPoint:TestPoint_THTPad_D1.5mm_Drill0.8mm" (id 2) (at 120.00 82.00 0) (effects (font (size 1.0 1.0)) hide))
     (property "Datasheet" "~" (id 3) (at 120.00 82.00 0) (effects (font (size 1.0 1.0)) hide))
@@
   (symbol (lib_id "RevC:TP1P") (at 140.00 82.00 0) (unit 1)
     (in_bom yes) (on_board yes)
-    (default_instance (reference "TP7") (unit 1) (value "GND") (footprint "TestPoint:TestPoint_THTPad_D1.5mm_Drill0.8mm"))
+    (default_instance (reference "TP7") (unit 1) (value "TP7") (footprint "TestPoint:TestPoint_THTPad_D1.5mm_Drill0.8mm"))
     (property "Reference" "TP7" (id 0) (at 140.00 79.00 0) (effects (font (size 1.0 1.0))))
-    (property "Value" "GND" (id 1) (at 140.00 85.00 0) (effects (font (size 0.9 0.9))))
+    (property "Value" "TP8" (id 1) (at 140.00 85.00 0) (effects (font (size 0.9 0.9))))
     (property "Footprint" "TestPoint:TestPoint_THTPad_D1.5mm_Drill0.8mm" (id 2) (at 140.00 82.00 0) (effects (font (size 1.0 1.0)) hide))
     (property "Datasheet" "~" (id 3) (at 140.00 82.00 0) (effects (font (size 1.0 1.0)) hide))
@@
   (symbol (lib_id "RevC:TP1P") (at 160.00 82.00 0) (unit 1)
     (in_bom yes) (on_board yes)
-    (default_instance (reference "TP8") (unit 1) (value "FLAG") (footprint "TestPoint:TestPoint_THTPad_D1.5mm_Drill0.8mm"))
+    (default_instance (reference "TP8") (unit 1) (value "TP8") (footprint "TestPoint:TestPoint_THTPad_D1.5mm_Drill0.8mm"))
     (property "Reference" "TP8" (id 0) (at 160.00 79.00 0) (effects (font (size 1.0 1.0))))
-    (property "Value" "FLAG" (id 1) (at 160.00 85.00 0) (effects (font (size 0.9 0.9))))
+    (property "Value" "TP8" (id 1) (at 160.00 85.00 0) (effects (font (size 0.9 0.9))))
     (property "Footprint" "TestPoint:TestPoint_THTPad_D1.5mm_Drill0.8mm" (id 2) (at 160.00 82.00 0) (effects (font (size 1.0 1.0)) hide))
     (property "Datasheet" "~" (id 3) (at 160.00 82.00 0) (effects (font (size 1.0 1.0)) hide))
@@
     (path "/612d3485-9937-4950-a59f-79d8ea9ecd9e" (reference "C106") (unit 1) (value "100n") (footprint "Capacitor_SMD:C_0805_2012Metric"))
     (path "/5b7d78e2-b83d-41f7-858b-07a036c8b157" (reference "C107") (unit 1) (value "10u 25V") (footprint "Capacitor_SMD:C_1206_3216Metric"))
-    (path "/2458628c-4d66-44bb-86c1-5a0473fa57c8" (reference "TP1") (unit 1) (value "TEST_A") (footprint "TestPoint:TestPoint_THTPad_D1.5mm_Drill0.8mm"))
-    (path "/736799eb-edd5-4b69-9ddd-91dad4e648ed" (reference "TP2") (unit 1) (value "OUT") (footprint "TestPoint:TestPoint_THTPad_D1.5mm_Drill0.8mm"))
-    (path "/d3d26d39-57a6-4fe0-a4bd-89bd6b5e923f" (reference "TP3") (unit 1) (value "NINV") (footprint "TestPoint:TestPoint_THTPad_D1.5mm_Drill0.8mm"))
-    (path "/1e35ef21-99ff-4d0a-bf2f-07446061f4b9" (reference "TP4") (unit 1) (value "INJ_NODE") (footprint "TestPoint:TestPoint_THTPad_D1.5mm_Drill0.8mm"))
-    (path "/18f6ff70-f5e9-471e-98ba-a9bbb35bc80e" (reference "TP5") (unit 1) (value "+12V") (footprint "TestPoint:TestPoint_THTPad_D1.5mm_Drill0.8mm"))
-    (path "/ac94ec31-bc7b-49b6-a0bd-485f1c75c87e" (reference "TP6") (unit 1) (value "-12V") (footprint "TestPoint:TestPoint_THTPad_D1.5mm_Drill0.8mm"))
-    (path "/f0017911-0819-4cc1-a520-9159d30924c5" (reference "TP7") (unit 1) (value "GND") (footprint "TestPoint:TestPoint_THTPad_D1.5mm_Drill0.8mm"))
-    (path "/5b2ca519-25af-41ec-a59d-abc5349957ef" (reference "TP8") (unit 1) (value "FLAG") (footprint "TestPoint:TestPoint_THTPad_D1.5mm_Drill0.8mm"))
+    (path "/2458628c-4d66-44bb-86c1-5a0473fa57c8" (reference "TP1") (unit 1) (value "TP1") (footprint "TestPoint:TestPoint_THTPad_D1.5mm_Drill0.8mm"))
+    (path "/736799eb-edd5-4b69-9ddd-91dad4e648ed" (reference "TP2") (unit 1) (value "TP2") (footprint "TestPoint:TestPoint_THTPad_D1.5mm_Drill0.8mm"))
+    (path "/d3d26d39-57a6-4fe0-a4bd-89bd6b5e923f" (reference "TP3") (unit 1) (value "TP3") (footprint "TestPoint:TestPoint_THTPad_D1.5mm_Drill0.8mm"))
+    (path "/1e35ef21-99ff-4d0a-bf2f-07446061f4b9" (reference "TP4") (unit 1) (value "TP4") (footprint "TestPoint:TestPoint_THTPad_D1.5mm_Drill0.8mm"))
+    (path "/18f6ff70-f5e9-471e-98ba-a9bbb35bc80e" (reference "TP5") (unit 1) (value "TP5") (footprint "TestPoint:TestPoint_THTPad_D1.5mm_Drill0.8mm"))
+    (path "/ac94ec31-bc7b-49b6-a0bd-485f1c75c87e" (reference "TP6") (unit 1) (value "TP6") (footprint "TestPoint:TestPoint_THTPad_D1.5mm_Drill0.8mm"))
+    (path "/f0017911-0819-4cc1-a520-9159d30924c5" (reference "TP7") (unit 1) (value "TP7") (footprint "TestPoint:TestPoint_THTPad_D1.5mm_Drill0.8mm"))
+    (path "/5b2ca519-25af-41ec-a59d-abc5349957ef" (reference "TP8") (unit 1) (value "TP8") (footprint "TestPoint:TestPoint_THTPad_D1.5mm_Drill0.8mm"))
   )
 )
